Commit message: feat(description): real kinematic measures from TFG2 system model
wheelbase=0.175, track=0.14, wheel_diameter=0.065 (fuente: memoria TFG2,
modelo del sistema). Anotados radio de giro min (0.175m) y velocidad
operativa (0.18 m/s) para la config de TEB/Nav2. Placeholders de
sensores reescalados al tamano real.

Co-Authored-By: Claude Fable 5 <noreply@anthropic.com>

File: src/robocar_description/urdf/robocar.urdf.xacro (robot description, xacro)
@@ -14,18 +14,22 @@
        Valores actuales = típicos de un chasis RC 1/10, solo orientativos.
        ══════════════════════════════════════════════════════════════════ -->
-  <!-- TODO(medir): distancia entre eje trasero y delantero (batalla) -->
-  <xacro:property name="wheelbase"      value="0.260"/>
-  <!-- TODO(medir): distancia entre centros de ruedas izq/der (via) -->
-  <xacro:property name="track_width"    value="0.180"/>
-  <!-- TODO(medir): diámetro de rueda / 2 -->
+  <!-- Batalla (L): 17.5 cm — fuente: memoria TFG2, modelo del sistema -->
+  <xacro:property name="wheelbase"      value="0.175"/>
+  <!-- Via (D): 14 cm — fuente: memoria TFG2, modelo del sistema -->
+  <xacro:property name="track_width"    value="0.140"/>
+  <!-- Ruedas de 6.5 cm de diametro — fuente: memoria TFG2 -->
   <xacro:property name="wheel_radius"   value="0.0325"/>
   <!-- TODO(medir): anchura de la rueda -->
-  <xacro:property name="wheel_width"    value="0.026"/>
+  <xacro:property name="wheel_width"    value="0.025"/>
   <!-- TODO(medir): largo x ancho x alto del chasis (caja aproximada) -->
-  <xacro:property name="chassis_length" value="0.360"/>
-  <xacro:property name="chassis_width"  value="0.190"/>
-  <xacro:property name="chassis_height" value="0.100"/>
+  <xacro:property name="chassis_length" value="0.280"/>
+  <xacro:property name="chassis_width"  value="0.150"/>
+  <xacro:property name="chassis_height" value="0.090"/>
   <!-- TODO(medir): cuanto sobresale el chasis por detras del eje trasero -->
   <xacro:property name="chassis_rear_overhang" value="0.050"/>
+  <!-- Otros datos del modelo del TFG2 (utiles para Nav2/TEB, no para el URDF):
+       angulo max de direccion ~45º -> radio de giro minimo = L/tan(45º) = 0.175 m
+       velocidad operativa probada = 0.18 m/s -->
+  <!-- Placeholders de sensores reescalados al tamano real del chasis -->
   <!-- Sensores: posicion respecto a base_link (centro eje trasero).
        x adelante, y izquierda, z arriba desde la altura del eje. -->
@@ -33,16 +37,16 @@
        de barrido sobre el eje). Si el conector USB queda hacia atras, dejar
        yaw=0; si no, ajustar la rotacion. -->
-  <xacro:property name="laser_x"   value="0.130"/>
-  <xacro:property name="laser_z"   value="0.120"/>
+  <xacro:property name="laser_x"   value="0.090"/>
+  <xacro:property name="laser_z"   value="0.110"/>
   <!-- TODO(medir): MPU6050 -->
-  <xacro:property name="imu_x"     value="0.100"/>
-  <xacro:property name="imu_z"     value="0.050"/>
+  <xacro:property name="imu_x"     value="0.070"/>
+  <xacro:property name="imu_z"     value="0.040"/>
   <!-- TODO(medir): camara USB frontal -->
-  <xacro:property name="camera_x"  value="0.300"/>
-  <xacro:property name="camera_z"  value="0.080"/>
+  <xacro:property name="camera_x"  value="0.200"/>
+  <xacro:property name="camera_z"  value="0.070"/>
   <!-- TODO(medir): ultrasonidos HC-SR04 frontales (centro y laterales) -->
-  <xacro:property name="us_x"      value="0.320"/>
-  <xacro:property name="us_y"      value="0.070"/>
-  <xacro:property name="us_z"      value="0.030"/>
+  <xacro:property name="us_x"      value="0.215"/>
+  <xacro:property name="us_y"      value="0.055"/>
+  <xacro:property name="us_z"      value="0.025"/>
   <!-- ══════════════ materiales (colores en Foxglove/RViz) ══════════════ -->
   <material name="body_grey"><color rgba="0.35 0.38 0.42 1"/></material>

Commit message: feat(description): measured chassis dimensions (35x17.5x13cm, overhang 8cm, wheel 2.6cm)
Co-Authored-By: Claude Fable 5 <noreply@anthropic.com>

File: src/robocar_description/urdf/robocar.urdf.xacro (robot description, xacro)
@@ -20,12 +20,13 @@
   <!-- Ruedas de 6.5 cm de diametro — fuente: memoria TFG2 -->
   <xacro:property name="wheel_radius"   value="0.0325"/>
-  <!-- TODO(medir): anchura de la rueda -->
-  <xacro:property name="wheel_width"    value="0.025"/>
-  <!-- TODO(medir): largo x ancho x alto del chasis (caja aproximada) -->
-  <xacro:property name="chassis_length" value="0.280"/>
-  <xacro:property name="chassis_width"  value="0.150"/>
-  <xacro:property name="chassis_height" value="0.090"/>
-  <!-- TODO(medir): cuanto sobresale el chasis por detras del eje trasero -->
-  <xacro:property name="chassis_rear_overhang" value="0.050"/>
+  <!-- Ancho de rueda: 2.6 cm (medido jul 2026) -->
+  <xacro:property name="wheel_width"    value="0.026"/>
+  <!-- Chasis (medido jul 2026): 35 cm largo x 17.5 cm ancho max x 13 cm de
+       alto DESDE EL SUELO (la caja parte de la altura del eje: 13 - 3.25) -->
+  <xacro:property name="chassis_length" value="0.350"/>
+  <xacro:property name="chassis_width"  value="0.175"/>
+  <xacro:property name="chassis_height" value="0.0975"/>
+  <!-- Voladizo trasero: 8 cm (medido jul 2026) -->
+  <xacro:property name="chassis_rear_overhang" value="0.080"/>
   <!-- Otros datos del modelo del TFG2 (utiles para Nav2/TEB, no para el URDF):
        angulo max de direccion ~45º -> radio de giro minimo = L/tan(45º) = 0.175 m

Commit message: feat(description): sensor positions measured (lidar, imu, 3x ultrasound); camera unmounted flag
LIDAR 7cm/6cm suelo (pendiente verificar 360 libres); IMU ~21cm/10cm;
ultrasonidos convertidos de referencia cola->cinta (central 27, lat 26,
y=+-5.25, z=7). Camara desmontada tras xacro:if camera_mounted.

Co-Authored-By: Claude Fable 5 <noreply@anthropic.com>

File: src/robocar_description/urdf/robocar.urdf.xacro (robot description, xacro)
@@ -38,16 +38,27 @@
        de barrido sobre el eje). Si el conector USB queda hacia atras, dejar
        yaw=0; si no, ajustar la rotacion. -->
-  <xacro:property name="laser_x"   value="0.090"/>
-  <xacro:property name="laser_z"   value="0.110"/>
-  <!-- TODO(medir): MPU6050 -->
-  <xacro:property name="imu_x"     value="0.070"/>
-  <xacro:property name="imu_z"     value="0.040"/>
-  <!-- TODO(medir): camara USB frontal -->
+  <!-- LIDAR (medido jul 2026): 7cm de la cinta, plano de barrido a 6cm del
+       suelo (rel. eje: 6 - 3.25). OJO: pendiente confirmar que el barrido
+       tiene 360 grados libres (el coche mide 13cm de alto). -->
+  <xacro:property name="laser_x"   value="0.070"/>
+  <xacro:property name="laser_z"   value="0.0275"/>
+  <!-- IMU (aprox jul 2026): ~21cm de la cinta (pendiente confirmar: la
+       descripcion decia "detras de las delanteras" = ~15-16), chip a 10cm
+       del suelo, centrado. -->
+  <xacro:property name="imu_x"     value="0.210"/>
+  <xacro:property name="imu_z"     value="0.0675"/>
+  <!-- Camara: DESMONTADA (jul 2026, mastil retirado). Reactivar con el flag
+       si vuelve el lane-following. -->
+  <xacro:property name="camera_mounted" value="false"/>
   <xacro:property name="camera_x"  value="0.200"/>
   <xacro:property name="camera_z"  value="0.070"/>
-  <!-- TODO(medir): ultrasonidos HC-SR04 frontales (centro y laterales) -->
-  <xacro:property name="us_x"      value="0.215"/>
-  <xacro:property name="us_y"      value="0.055"/>
-  <xacro:property name="us_z"      value="0.025"/>
+  <!-- Ultrasonidos (medidos jul 2026 DESDE LA COLA; convertidos a cinta
+       restando el voladizo de 8cm): central en el morro (27cm), laterales
+       1cm retranqueados (26cm) y a 3.5cm del borde -> y=+-5.25cm. Altura
+       7cm del suelo (rel. eje: 7 - 3.25). -->
+  <xacro:property name="us_x"      value="0.270"/>
+  <xacro:property name="us_side_x" value="0.260"/>
+  <xacro:property name="us_y"      value="0.0525"/>
+  <xacro:property name="us_z"      value="0.0375"/>
   <!-- ══════════════ materiales (colores en Foxglove/RViz) ══════════════ -->
   <material name="body_grey"><color rgba="0.35 0.38 0.42 1"/></material>
@@ -116,18 +127,20 @@
     <origin xyz="${imu_x} 0 ${imu_z}"/>
   </joint>
-  <!-- Cámara frontal -->
-  <link name="camera_link">
-    <visual>
-      <geometry><box size="0.025 0.06 0.025"/></geometry>
-      <material name="sensor_blue"/>
-    </visual>
-  </link>
-  <joint name="camera_joint" type="fixed">
-    <parent link="base_link"/>
-    <child link="camera_link"/>
-    <origin xyz="${camera_x} 0 ${camera_z}"/>
-  </joint>
+  <!-- Cámara frontal (desmontada; se incluye solo si camera_mounted=true) -->
+  <xacro:if value="${camera_mounted}">
+    <link name="camera_link">
+      <visual>
+        <geometry><box size="0.025 0.06 0.025"/></geometry>
+        <material name="sensor_blue"/>
+      </visual>
+    </link>
+    <joint name="camera_joint" type="fixed">
+      <parent link="base_link"/>
+      <child link="camera_link"/>
+      <origin xyz="${camera_x} 0 ${camera_z}"/>
+    </joint>
+  </xacro:if>
   <!-- Ultrasonidos HC-SR04 (izq / centro / der), apuntando hacia delante -->
-  <xacro:macro name="ultrasound" params="name y">
+  <xacro:macro name="ultrasound" params="name x y">
     <link name="${name}">
       <visual>
@@ -139,9 +152,9 @@
       <parent link="base_link"/>
       <child link="${name}"/>
-      <origin xyz="${us_x} ${y} ${us_z}"/>
+      <origin xyz="${x} ${y} ${us_z}"/>
     </joint>
   </xacro:macro>
-  <xacro:ultrasound name="ultrasound_left"   y="${us_y}"/>
-  <xacro:ultrasound name="ultrasound_center" y="0"/>
-  <xacro:ultrasound name="ultrasound_right"  y="${-us_y}"/>
+  <xacro:ultrasound name="ultrasound_left"   x="${us_side_x}" y="${us_y}"/>
+  <xacro:ultrasound name="ultrasound_center" x="${us_x}"      y="0"/>
+  <xacro:ultrasound name="ultrasound_right"  x="${us_side_x}" y="${-us_y}"/>
 </robot>

Commit message: feat(description): confirmed sensor measures (us 25/24cm from axle, imu 21, overhang 8.5)
LIDAR: posible oclusion solo en sector trasero (radiador RPi sobre eje);
verificar con /scan en Foxglove, filtrar o elevar si molesta.

Co-Authored-By: Claude Fable 5 <noreply@anthropic.com>

File: src/robocar_description/urdf/robocar.urdf.xacro (robot description, xacro)
@@ -27,6 +27,6 @@
   <xacro:property name="chassis_width"  value="0.175"/>
   <xacro:property name="chassis_height" value="0.0975"/>
-  <!-- Voladizo trasero: 8 cm (medido jul 2026) -->
-  <xacro:property name="chassis_rear_overhang" value="0.080"/>
+  <!-- Voladizo trasero: 8.5-9 cm (medido jul 2026) -->
+  <xacro:property name="chassis_rear_overhang" value="0.085"/>
   <!-- Otros datos del modelo del TFG2 (utiles para Nav2/TEB, no para el URDF):
        angulo max de direccion ~45º -> radio de giro minimo = L/tan(45º) = 0.175 m
@@ -38,12 +38,12 @@
        de barrido sobre el eje). Si el conector USB queda hacia atras, dejar
        yaw=0; si no, ajustar la rotacion. -->
-  <!-- LIDAR (medido jul 2026): 7cm de la cinta, plano de barrido a 6cm del
-       suelo (rel. eje: 6 - 3.25). OJO: pendiente confirmar que el barrido
-       tiene 360 grados libres (el coche mide 13cm de alto). -->
+  <!-- LIDAR (medido jul 2026): 7cm del eje trasero, plano de barrido a 6cm
+       del suelo (rel. eje: 6 - 3.25). Posible oclusion SOLO en el sector
+       trasero (radiador de la RPi sobre el eje): verificar con /scan en
+       Foxglove y filtrar sector o elevar el LIDAR si molesta. -->
   <xacro:property name="laser_x"   value="0.070"/>
   <xacro:property name="laser_z"   value="0.0275"/>
-  <!-- IMU (aprox jul 2026): ~21cm de la cinta (pendiente confirmar: la
-       descripcion decia "detras de las delanteras" = ~15-16), chip a 10cm
-       del suelo, centrado. -->
+  <!-- IMU (confirmado jul 2026): 21-22cm del eje trasero, chip a 10cm del
+       suelo, centrado. -->
   <xacro:property name="imu_x"     value="0.210"/>
   <xacro:property name="imu_z"     value="0.0675"/>
@@ -53,10 +53,9 @@
   <xacro:property name="camera_x"  value="0.200"/>
   <xacro:property name="camera_z"  value="0.070"/>
-  <!-- Ultrasonidos (medidos jul 2026 DESDE LA COLA; convertidos a cinta
-       restando el voladizo de 8cm): central en el morro (27cm), laterales
-       1cm retranqueados (26cm) y a 3.5cm del borde -> y=+-5.25cm. Altura
-       7cm del suelo (rel. eje: 7 - 3.25). -->
-  <xacro:property name="us_x"      value="0.270"/>
-  <xacro:property name="us_side_x" value="0.260"/>
+  <!-- Ultrasonidos (confirmados jul 2026, medidos desde el eje trasero):
+       central a 25cm, laterales 1cm retranqueados (24cm) y a 3.5cm del
+       borde -> y=+-5.25cm. Altura 7cm del suelo (rel. eje: 7 - 3.25). -->
+  <xacro:property name="us_x"      value="0.250"/>
+  <xacro:property name="us_side_x" value="0.240"/>
   <xacro:property name="us_y"      value="0.0525"/>
   <xacro:property name="us_z"      value="0.0375"/>

Commit message: fix(viz): energy readings are reliable (Ruben); angled side ultrasounds (~25deg TODO confirm)
Co-Authored-By: Claude Fable 5 <noreply@anthropic.com>

File: src/robocar_description/urdf/robocar.urdf.xacro (robot description, xacro)
@@ -140,6 +140,8 @@
     </joint>
   </xacro:if>
-  <!-- Ultrasonidos HC-SR04 (izq / centro / der), apuntando hacia delante -->
-  <xacro:macro name="ultrasound" params="name x y">
+  <!-- Ultrasonidos HC-SR04 (izq / centro / der). Los laterales miran hacia
+       afuera ~25 grados (TODO confirmar angulo exacto). -->
+  <xacro:property name="us_yaw" value="0.436"/>
+  <xacro:macro name="ultrasound" params="name x y yaw">
     <link name="${name}">
       <visual>
@@ -151,9 +153,9 @@
       <parent link="base_link"/>
       <child link="${name}"/>
-      <origin xyz="${x} ${y} ${us_z}"/>
+      <origin xyz="${x} ${y} ${us_z}" rpy="0 0 ${yaw}"/>
     </joint>
   </xacro:macro>
-  <xacro:ultrasound name="ultrasound_left"   x="${us_side_x}" y="${us_y}"/>
-  <xacro:ultrasound name="ultrasound_center" x="${us_x}"      y="0"/>
-  <xacro:ultrasound name="ultrasound_right"  x="${us_side_x}" y="${-us_y}"/>
+  <xacro:ultrasound name="ultrasound_left"   x="${us_side_x}" y="${us_y}"  yaw="${us_yaw}"/>
+  <xacro:ultrasound name="ultrasound_center" x="${us_x}"      y="0"        yaw="0"/>
+  <xacro:ultrasound name="ultrasound_right"  x="${us_side_x}" y="${-us_y}" yaw="${-us_yaw}"/>
 </robot>

Commit message: fix(lidar): C1 zero-angle points backwards with current mount — 180deg yaw on laser frame
Verificado contra los ultrasonidos: el escaneo se dibujaba girado 180
(la 'pared' frontal era en realidad trasera). Fix en URDF (hereda a
Cartographer/Nav2) y en el panel.

Co-Authored-By: Claude Fable 5 <noreply@anthropic.com>

File: src/robocar_description/urdf/robocar.urdf.xacro (robot description, xacro)
@@ -109,8 +109,11 @@
     </visual>
   </link>
+  <!-- El 0 grados del RPLidar C1 apunta HACIA ATRAS con el montaje actual
+       (flecha del sensor hacia las ruedas delanteras) -> giro de 180 en yaw.
+       Verificado empiricamente contra los ultrasonidos (jul 2026). -->
   <joint name="laser_joint" type="fixed">
     <parent link="base_link"/>
     <child link="laser"/>
-    <origin xyz="${laser_x} 0 ${laser_z}" rpy="0 0 0"/>
+    <origin xyz="${laser_x} 0 ${laser_z}" rpy="0 0 ${pi}"/>
   </joint>
   <!-- IMU: frame "imu_link" (usarlo en accelerometer_node, hito 0.5) -->

Commit message: fix(urdf): base_link como raiz (base_footprint hijo) -> arbol TF unico para Nav2
base_footprint_joint invertido: parent=base_link, child=base_footprint, z=-wheel_radius. Antes base_footprint era padre de base_link y ademas la odometria publica odom->base_link => base_link con dos padres => arbol partido (odom->base_footprint daba two unconnected trees). Ahora odom->base_link->{base_footprint,laser,...} unico. Verificado: odom->base_footprint [0,0,-0.033] resuelve, odom->laser [0.070,0,0.028]+180deg ok. Coherente con base_link_frame=base_link (EKF) y robot_base_frame=base_link (Nav2).

Co-Authored-By: Claude Opus 4.8 (1M context) <noreply@anthropic.com>

File: src/robocar_description/urdf/robocar.urdf.xacro (robot description, xacro)
@@ -93,7 +93,7 @@
   </link>
   <joint name="base_footprint_joint" type="fixed">
-    <parent link="base_footprint"/>
-    <child link="base_link"/>
-    <origin xyz="0 0 ${wheel_radius}"/>
+    <parent link="base_link"/>
+    <child link="base_footprint"/>
+    <origin xyz="0 0 ${-wheel_radius}"/>
   </joint>
   <!-- ruedas -->
